File: kicad/radar_5g8_fe/radar_5g8_fe.kicad_pcb (KiCad board)
At the start: 4 copper layers, 100 x 100 mm, 127 parts, among them J5 8x2 2.54 mm header, Q3 AO3401A, Q4 2N7002

Commit message: Auto-update: 2026-08-09 20:12:01
Parts:
- removed FID22_97, FID78_97: , 
- removed H52_15, H52_84, H63_43, H63_57: M3, 
- added FID6_97: , , F.Cu at (6.00, 3.00)
- added FID94_97: , , F.Cu at (94.0, 3.00)
- added H52_16: M3, , F.Cu at (52.0, 83.2)
- added H52_83: M3, , F.Cu at (52.0, 16.8)
- added H63_29: M3, , F.Cu at (63.0, 71.0)
- added H63_71: M3, , F.Cu at (63.0, 29.0)
- moved CAD0 2.50 mm to (87.9, 84.2)
- moved CAD2 2.50 mm to (84.5, 84.2)
- moved CBD0 2.50 mm to (87.9, 15.8)
- moved CBD2 2.50 mm to (84.5, 15.8)
- moved DA1 2.50 mm to (89.7, 84.2)
- moved DB1 2.50 mm to (89.7, 15.8)
- moved RAD1 2.50 mm to (86.2, 84.2)
- moved RAO 2.50 mm to (82.7, 84.2)
- moved RAT 2.50 mm to (93.7, 84.2)
- moved RBD1 2.50 mm to (86.2, 15.8)
- moved RBO 2.50 mm to (82.7, 15.8)
- moved RBT 2.50 mm to (93.7, 15.8)
- moved CA93 1.80 mm to (46.4, 80.6)
- moved CB93 1.80 mm to (46.4, 19.4)
- moved CA5 1.50 mm to (36.0, 78.3)
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Routing:
- net GND: vias 695 -> 680
- net EN: vias 3 -> 2

Commit message: Auto-update: 2026-08-09 20:14:38
Parts:
- removed H52_16, H52_83: M3, 
- added H54_16: M3, , F.Cu at (54.0, 83.2)
- added H54_83: M3, , F.Cu at (54.0, 16.8)
- added TP1: thermal face, , F.Cu at (52.0, 92.0)
- added TP2: thermal face, , F.Cu at (34.0, 92.0)
- added TP3: thermal face, , F.Cu at (52.0, 8.00)
- added TP4: thermal face, , F.Cu at (34.0, 8.00)
- added TP5: thermal face, , F.Cu at (59.5, 64.0)
- added TP6: thermal face, , F.Cu at (59.5, 36.0)
- moved RCF 2.50 mm to (37.0, 59.6)
- moved RDF 2.50 mm to (37.0, 40.4)
Routing:
- net GND: vias 680 -> 682

Commit message: Auto-update: 2026-08-09 20:16:17
Parts:
- removed H54_16, H54_83, H63_29, H63_71: M3, 
- added H19_3: M3, , F.Cu at (19.5, 96.5)
- added H19_96: M3, , F.Cu at (19.5, 3.50)
- added H44_3: M3, , F.Cu at (44.0, 96.5)
- added H44_96: M3, , F.Cu at (44.0, 3.50)
- TP1, TP2, TP3, TP4, TP5, TP6: moved to B.Cu
- turned TP1 to 180 degrees
- turned TP2 to 180 degrees
- turned TP3 to 180 degrees
- turned TP4 to 180 degrees
- turned TP5 to 180 degrees
- turned TP6 to 180 degrees
Routing:
- net GND: vias 682 -> 692
