File: kicad/radar_5g8_receive_array/radar_5g8_receive.kicad_pcb (KiCad board)
At the start: 2 copper layers, 47.2 x 71.3 mm, 11 parts

Commit message: Auto-update: 2026-08-09 20:18:09
Parts:
- moved H1 1.03 mm to (4.00, 27.4)
- moved H5 1.03 mm to (13.0, 36.4)
- moved R3 0.93 mm to (5.85, 55.9)
- moved R4 0.93 mm to (5.85, 5.90)
- moved D2 0.51 mm to (7.00, 17.7)
- moved D1 0.50 mm to (7.00, 67.8)
Other:
- board size 47.2 x 71.3 mm -> 47.2 x 71.4 mm
- board text added: "ABSORBER BETWEEN THE BOARDS"
- board text added: "MOUNT >= 200 mm APART"
