File: kicad/radar_5g8_receive_array/radar_5g8_receive.kicad_pcb (KiCad board)
At the start: 2 copper layers, 47.2 x 71.4 mm, 11 parts

Commit message: Auto-update: 2026-08-09 20:24:15
Parts:
- D1, D2: footprint radar5g8:D_0402_Limiter -> radar5g8:D_0805_Limiter
- R3, R4: footprint radar5g8:R_0402_50R -> radar5g8:R_0805_1W_50R
