File: kicad/radar_5g8_receive_array/radar_5g8_receive.kicad_pcb (KiCad board)
At the start: 2 copper layers, 47.2 x 71.4 mm, 11 parts

Commit message: Auto-update: 2026-08-09 20:44:04
Parts:
- removed H4, H5: M3, radar5g8:MountingHole_M3
- moved H3 40.5 mm to (17.0, 35.4)
- moved H2 40.3 mm to (8.00, 47.4)
Routing:
- net GND: vias 16 -> 18
