File: kicad/radar_5g8_transmit_array/radar_5g8_transmit.kicad_pcb (KiCad board)
At the start: 2 copper layers, 71.3 x 47.2 mm, 9 parts

Commit message: Auto-update: 2026-08-09 20:18:09
Parts:
- removed H5: M3, radar5g8:MountingHole_M3
- moved H2 63.1 mm to (67.0, 7.24)
- moved H1 57.3 mm to (4.00, 4.24)
- moved H3 51.1 mm to (34.0, 43.2)
- moved H4 16.8 mm to (40.0, 34.2)
- moved R1 0.93 mm to (15.4, 41.4)
- moved R2 0.93 mm to (65.4, 41.4)
Other:
- board text added: "ABSORBER BETWEEN THE BOARDS"
- board text added: "MOUNT >= 200 mm APART"
