File: kicad/radar_5g8_transmit_array/radar_5g8_transmit.kicad_pcb (KiCad board)
At the start: 2 copper layers, 71.3 x 47.2 mm, 8 parts

Commit message: Auto-update: 2026-08-09 20:24:15
Parts:
- R1, R2: footprint radar5g8:R_0402_50R -> radar5g8:R_0805_1W_50R
Changed lines of the file:
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@@
-		(embedded_fonts no)
-	)
-	(footprint "radar5g8:R_0402_50R"
-		(layer "F.Cu")
-		(at 15.398231 41.386984 90)
-		(property "Reference" "R1"
-			(at 0 0 90)
-			(layer "F.SilkS")
-			(hide yes)
-			(effects
-				(font
-					(size 1.27 1.27)
-				)
-			)
-		)
-		(property "Value" "50R"
-			(at 0 0 90)
-			(layer "F.Fab")
-			(hide yes)
-			(effects
-				(font
-					(size 1.27 1.27)
-				)
-			)
-		)
-		(property "Datasheet" ""
-			(at 0 0 90)
-			(layer "F.Fab")
-			(hide yes)
-			(effects
-				(font
-					(size 1.27 1.27)
-				)
-			)
-		)
-		(property "Description" ""
-			(at 0 0 90)
-			(layer "F.Fab")
-			(hide yes)
-			(effects
-				(font
-					(size 1.27 1.27)
-				)
-			)
-		)
-		(attr smd)
-		(duplicate_pad_numbers_are_jumpers no)
-		(fp_rect
-			(start 1.609999 -0.56)
-			(end -1.609999 0.56)
-			(stroke
-				(width 0.05)
-				(type default)
-			)
-			(fill no)
-			(layer "F.CrtYd")
-		)
-		(pad "1" smd rect
-			(at 1.049999 0 90)
-			(size 0.62 0.62)
-			(layers "F.Cu" "F.Mask" "F.Paste")
-			(net "TX1")
-			(thermal_bridge_angle 45)
-		)
-		(pad "2" smd rect
-			(at -1.049999 0 90)
-			(size 0.62 0.62)
-			(layers "F.Cu" "F.Mask" "F.Paste")
-			(net "GND")
-			(thermal_bridge_angle 45)
-		)
 		(embedded_fonts no)
 	)
@@
 	(footprint "radar5g8:MountingHole_M3"
 		(layer "F.Cu")
-		(at 4 4.237)
-		(property "Reference" "H1"
+		(at 67 7.237)
+		(property "Reference" "H2"
 			(at 0 0 0)
 			(layer "F.SilkS")
@@
 		(embedded_fonts no)
 	)
-	(footprint "radar5g8:R_0402_50R"
-		(layer "F.Cu")
-		(at 65.442137 41.386984 90)
-		(property "Reference" "R2"
+	(footprint "radar5g8:R_0805_1W_50R"
+		(layer "F.Cu")
+		(at 15.398231 41.386984 90)
+		(property "Reference" "R1"
 			(at 0 0 90)
 			(layer "F.SilkS")
@@
 		(duplicate_pad_numbers_are_jumpers no)
 		(fp_rect
-			(start 1.609999 -0.56)
-			(end -1.609999 0.56)
+			(start 1.949999 -0.75)
+			(end -1.949999 0.75)
 			(stroke
 				(width 0.05)
@@
 		(pad "1" smd rect
 			(at 1.049999 0 90)
-			(size 0.62 0.62)
+			(size 1 1.3)
+			(layers "F.Cu" "F.Mask" "F.Paste")
+			(net "TX1")
+			(thermal_bridge_angle 45)
+		)
+		(pad "2" smd rect
+			(at -1.049999 0 90)
+			(size 1 1.3)
+			(layers "F.Cu" "F.Mask" "F.Paste")
+			(net "GND")
+			(thermal_bridge_angle 45)
+		)
+		(embedded_fonts no)
+	)
+	(footprint "radar5g8:SMA_EndLaunch_50R_BottomEdge"
+		(layer "F.Cu")
+		(at 56.443906 47.237)
+		(property "Reference" "TX2"
+			(at 0 0 0)
+			(layer "F.SilkS")
+			(hide yes)
+			(effects
+				(font
+					(size 1.27 1.27)
+				)
+			)
+		)
+		(property "Value" "SMA-EDGE-50R"
+			(at 0 0 0)
+			(layer "F.Fab")
+			(hide yes)
+			(effects
+				(font
+					(size 1.27 1.27)
+				)
+			)
+		)
+		(property "Datasheet" ""
+			(at 0 0 0)
+			(layer "F.Fab")
+			(hide yes)
+			(effects
+				(font
+					(size 1.27 1.27)
+				)
+			)
+		)
+		(property "Description" ""
+			(at 0 0 0)
+			(layer "F.Fab")
+			(hide yes)
+			(effects
+				(font
+					(size 1.27 1.27)
+				)
+			)
+		)
+		(duplicate_pad_numbers_are_jumpers no)
+		(fp_rect
+			(start -4.946664 -3.3)
+			(end 4.946664 0.1)
+			(stroke
+				(width 0.05)
+				(type default)
+			)
+			(fill no)
+			(layer "F.CrtYd")
+		)
+		(pad "1" smd rect
+			(at 0 -1.3)
+			(size 1.853528 2.3)
 			(layers "F.Cu" "F.Mask" "F.Paste")
 			(net "TX2")
@@
 		)
 		(pad "2" smd rect
-			(at -1.049999 0 90)
-			(size 0.62 0.62)
+			(at -3.396664 -1.6)
+			(size 2.6 2.9)
 			(layers "F.Cu" "F.Mask" "F.Paste")
 			(net "GND")
 			(thermal_bridge_angle 45)
 		)
+		(pad "3" smd rect
+			(at 3.396664 -1.6)
+			(size 2.6 2.9)
+			(layers "F.Cu" "F.Mask" "F.Paste")
+			(net "GND")
+			(thermal_bridge_angle 45)
+		)
 		(embedded_fonts no)
 	)
 	(footprint "radar5g8:MountingHole_M3"
 		(layer "F.Cu")
-		(at 34 43.237)
-		(property "Reference" "H3"
+		(at 4 4.237)
+		(property "Reference" "H1"
 			(at 0 0 0)
 			(layer "F.SilkS")
@@
 	(footprint "radar5g8:MountingHole_M3"
 		(layer "F.Cu")
-		(at 67 7.237)
-		(property "Reference" "H2"
+		(at 34 43.237)
+		(property "Reference" "H3"
 			(at 0 0 0)
 			(layer "F.SilkS")
@@
 		(embedded_fonts no)
 	)
-	(footprint "radar5g8:SMA_EndLaunch_50R_BottomEdge"
-		(layer "F.Cu")
-		(at 56.443906 47.237)
-		(property "Reference" "TX2"
-			(at 0 0 0)
+	(footprint "radar5g8:R_0805_1W_50R"
+		(layer "F.Cu")
+		(at 65.442137 41.386984 90)
+		(property "Reference" "R2"
+			(at 0 0 90)
 			(layer "F.SilkS")
 			(hide yes)
@@
 			)
 		)
-		(property "Value" "SMA-EDGE-50R"
-			(at 0 0 0)
+		(property "Value" "50R"
+			(at 0 0 90)
 			(layer "F.Fab")
 			(hide yes)
@@
 		)
 		(property "Datasheet" ""
-			(at 0 0 0)
+			(at 0 0 90)
 			(layer "F.Fab")
 			(hide yes)
@@
 		)
 		(property "Description" ""
-			(at 0 0 0)
-			(layer "F.Fab")
-			(hide yes)
-			(effects
-				(font
-					(size 1.27 1.27)
-				)
-			)
-		)
+			(at 0 0 90)
+			(layer "F.Fab")
+			(hide yes)
+			(effects
+				(font
+					(size 1.27 1.27)
+				)
+			)
+		)
+		(attr smd)
 		(duplicate_pad_numbers_are_jumpers no)
 		(fp_rect
-			(start -4.946664 -3.3)
-			(end 4.946664 0.1)
+			(start 1.949999 -0.75)
+			(end -1.949999 0.75)
 			(stroke
 				(width 0.05)
@@
 		)
 		(pad "1" smd rect
-			(at 0 -1.3)
-			(size 1.853528 2.3)
+			(at 1.049999 0 90)
+			(size 1 1.3)
 			(layers "F.Cu" "F.Mask" "F.Paste")
 			(net "TX2")
@@
 		)
 		(pad "2" smd rect
-			(at -3.396664 -1.6)
-			(size 2.6 2.9)
-			(layers "F.Cu" "F.Mask" "F.Paste")
-			(net "GND")
-			(thermal_bridge_angle 45)
-		)
-		(pad "3" smd rect
-			(at 3.396664 -1.6)
-			(size 2.6 2.9)
+			(at -1.049999 0 90)
+			(size 1 1.3)
 			(layers "F.Cu" "F.Mask" "F.Paste")
 			(net "GND")
@@
 	)
 	(via
+		(at 9.146664 44.767)
+		(size 0.75)
+		(drill 0.4)
+		(layers "F.Cu" "B.Cu")
+		(net "GND")
+	)
+	(via
 		(at 53.697242 44.767)
 		(size 0.75)
@@
 	)
 	(via
+		(at 66.192137 43.686984)
+		(size 0.75)
+		(drill 0.4)
+		(layers "F.Cu" "B.Cu")
+		(net "GND")
+	)
+	(via
+		(at 3.653336 46.037)
+		(size 0.75)
+		(drill 0.4)
+		(layers "F.Cu" "B.Cu")
+		(net "GND")
+	)
+	(via
+		(at 59.19057 46.037)
+		(size 0.75)
+		(drill 0.4)
+		(layers "F.Cu" "B.Cu")
+		(net "GND")
+	)
+	(via
+		(at 9.146664 46.037)
+		(size 0.75)
+		(drill 0.4)
+		(layers "F.Cu" "B.Cu")
+		(net "GND")
+	)
+	(via
+		(at 48.17099 44.387)
+		(size 0.75)
+		(drill 0.4)
+		(layers "F.Cu" "B.Cu")
+		(net "GND")
+	)
+	(via
+		(at 14.648231 43.686984)
+		(size 0.75)
+		(drill 0.4)
+		(layers "F.Cu" "B.Cu")
+		(net "GND")
+	)
+	(via
+		(at 53.697242 46.037)
+		(size 0.75)
+		(drill 0.4)
+		(layers "F.Cu" "B.Cu")
+		(net "GND")
+	)
+	(via
+		(at 59.19057 44.767)
+		(size 0.75)
+		(drill 0.4)
+		(layers "F.Cu" "B.Cu")
+		(net "GND")
+	)
+	(via
+		(at 3.653336 44.767)
+		(size 0.75)
+		(drill 0.4)
+		(layers "F.Cu" "B.Cu")
+		(net "GND")
+	)
+	(via
 		(at 16.148231 43.686984)
 		(size 0.75)
@@
 	)
 	(via
-		(at 59.19057 44.767)
-		(size 0.75)
-		(drill 0.4)
-		(layers "F.Cu" "B.Cu")
-		(net "GND")
-	)
-	(via
-		(at 59.19057 46.037)
-		(size 0.75)
-		(drill 0.4)
-		(layers "F.Cu" "B.Cu")
-		(net "GND")
-	)
-	(via
-		(at 9.146664 46.037)
-		(size 0.75)
-		(drill 0.4)
-		(layers "F.Cu" "B.Cu")
-		(net "GND")
-	)
-	(via
 		(at 23.17099 44.387)
 		(size 0.75)
@@
 	)
 	(via
-		(at 14.648231 43.686984)
-		(size 0.75)
-		(drill 0.4)
-		(layers "F.Cu" "B.Cu")
-		(net "GND")
-	)
-	(via
-		(at 53.697242 46.037)
-		(size 0.75)
-		(drill 0.4)
-		(layers "F.Cu" "B.Cu")
-		(net "GND")
-	)
-	(via
-		(at 9.146664 44.767)
-		(size 0.75)
-		(drill 0.4)
-		(layers "F.Cu" "B.Cu")
-		(net "GND")
-	)
-	(via
-		(at 3.653336 44.767)
-		(size 0.75)
-		(drill 0.4)
-		(layers "F.Cu" "B.Cu")
-		(net "GND")
-	)
-	(via
 		(at 64.692137 43.686984)
 		(size 0.75)
 		(drill 0.4)
-		(layers "F.Cu" "B.Cu")
-		(net "GND")
-	)
-	(via
-		(at 3.653336 46.037)
-		(size 0.75)
-		(drill 0.4)
-		(layers "F.Cu" "B.Cu")
-		(net "GND")
-	)
-	(via
-		(at 48.17099 44.387)
-		(size 0.75)
-		(drill 0.4)
-		(layers "F.Cu" "B.Cu")
-		(net "GND")
-	)
-	(via
-		(at 66.192137 43.686984)
-		(size 0.75)
-		(drill 0.4)
