File: kicad/radar_5g8_transmit_array/radar_5g8_transmit.kicad_pcb (KiCad board)
At the start: 2 copper layers, 71.3 x 47.2 mm, 8 parts

Commit message: Auto-update: 2026-08-09 20:43:43
Parts:
- added H5: M3, radar5g8:MountingHole_M3, F.Cu at (29.0, 30.2)
- moved H4 5.00 mm to (43.0, 30.2)
