File: kicad/radar_5g8_lna/radar_5g8_lna.kicad_pcb (KiCad board)
At the start: 4 copper layers, 92 x 68 mm, 82 parts, among them J5 2x7 2.54 mm header, Q3 AO3401A, Q4 2N7002

Commit message: Auto-update: 2026-08-09 20:21:04
Parts:
- added TP1: thermal face, , B.Cu at (38.0, 10.0)
- added TP2: thermal face, , B.Cu at (38.0, 58.0)
