File: kicad/radar_5g8_pa/radar_5g8_pa.kicad_pcb (KiCad board)
At the start: 4 copper layers, 100 x 84 mm, 85 parts, among them J5 2x7 2.54 mm header, Q3 AO3401A, Q4 2N7002

Commit message: Auto-update: 2026-08-09 20:21:04
Parts:
- added TP1: thermal face, , B.Cu at (40.5, 10.0)
- added TP2: thermal face, , B.Cu at (22.5, 10.0)
- added TP3: thermal face, , B.Cu at (40.5, 74.0)
- added TP4: thermal face, , B.Cu at (22.5, 74.0)
